File: output/pcbs/wings.kicad_pcb (KiCad board)
At the start: 2 copper layers, 147.9 x 119.9 mm, 60 parts

Commit message: add all ergogen outputs
Connections:
- MCUF1 pad 15: GND -> VIN
- MCUF1 pad 16: VIN -> GND
- S27 pad 1: P2 -> P4
- S29 pad 1: P1 -> P5
Changed lines of the file:
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@@
   (title_block
     (title "wings")
-    (date "2024-11-10")
+    (date "2024-11-27")
     (rev "0.1")
     (company "lad1337")
@@
             (fp_text reference "S27" (at 0 0) (layer F.SilkS) (effects (font (size 1.27 1.27) (thickness 0.15))))
             (fp_text value "" (at 0 0) (layer F.SilkS) hide (effects (font (size 1.27 1.27) (thickness 0.15))))
-            (pad 1 smd rect (at 0 1.5 -30) (size 0.2 0.2) (layers F.Cu F.Paste F.Mask) (net 6 "P2"))
+            (pad 1 smd rect (at 0 1.5 -30) (size 0.2 0.2) (layers F.Cu F.Paste F.Mask) (net 26 "P4"))
             (pad 2 smd rect (at 0 2.5 -30) (size 0.2 0.2) (layers F.Cu F.Paste F.Mask) (net 33 "home_top"))
             (pad 3 smd rect (at 0 3.5 -30) (size 0.2 0.2) (layers F.Cu F.Paste F.Mask) (net 0 ""))
@@
             (fp_text reference "S29" (at 0 0) (layer F.SilkS) (effects (font (size 1.27 1.27) (thickness 0.15))))
             (fp_text value "" (at 0 0) (layer F.SilkS) hide (effects (font (size 1.27 1.27) (thickness 0.15))))
-            (pad 1 smd rect (at 0 1.5 -30) (size 0.2 0.2) (layers F.Cu F.Paste F.Mask) (net 11 "P1"))
+            (pad 1 smd rect (at 0 1.5 -30) (size 0.2 0.2) (layers F.Cu F.Paste F.Mask) (net 21 "P5"))
             (pad 2 smd rect (at 0 2.5 -30) (size 0.2 0.2) (layers F.Cu F.Paste F.Mask) (net 35 "far_top"))
             (pad 3 smd rect (at 0 3.5 -30) (size 0.2 0.2) (layers F.Cu F.Paste F.Mask) (net 0 ""))
@@
             (pad 13 smd rect (at 0 13.5 180) (size 0.2 0.2) (layers F.Cu F.Paste F.Mask) (net 42 "GND"))
             (pad 14 smd rect (at 0 14.5 180) (size 0.2 0.2) (layers F.Cu F.Paste F.Mask) (net 43 "5V"))
-            (pad 15 smd rect (at 0 15.5 180) (size 0.2 0.2) (layers F.Cu F.Paste F.Mask) (net 42 "GND"))
-            (pad 16 smd rect (at 0 16.5 180) (size 0.2 0.2) (layers F.Cu F.Paste F.Mask) (net 44 "VIN"))
+            (pad 15 smd rect (at 0 15.5 180) (size 0.2 0.2) (layers F.Cu F.Paste F.Mask) (net 44 "VIN"))
+            (pad 16 smd rect (at 0 16.5 180) (size 0.2 0.2) (layers F.Cu F.Paste F.Mask) (net 42 "GND"))
             (pad 17 smd rect (at 0 17.5 180) (size 0.2 0.2) (layers F.Cu F.Paste F.Mask) (net 45 "SWCLK"))
             (pad 18 smd rect (at 0 18.5 180) (size 0.2 0.2) (layers F.Cu F.Paste F.Mask) (net 46 "SWDIO"))

Commit message: switch keys for thumbs for easier tracing
Connections:
- S27 pad 1: P4 -> P5
- S29 pad 1: P5 -> P4
Changed lines of the file:
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@@
   (title_block
     (title "wings")
-    (date "2024-11-27")
+    (date "2024-11-28")
     (rev "0.1")
     (company "lad1337")
@@
             (fp_text reference "S27" (at 0 0) (layer F.SilkS) (effects (font (size 1.27 1.27) (thickness 0.15))))
             (fp_text value "" (at 0 0) (layer F.SilkS) hide (effects (font (size 1.27 1.27) (thickness 0.15))))
-            (pad 1 smd rect (at 0 1.5 -30) (size 0.2 0.2) (layers F.Cu F.Paste F.Mask) (net 26 "P4"))
+            (pad 1 smd rect (at 0 1.5 -30) (size 0.2 0.2) (layers F.Cu F.Paste F.Mask) (net 21 "P5"))
             (pad 2 smd rect (at 0 2.5 -30) (size 0.2 0.2) (layers F.Cu F.Paste F.Mask) (net 33 "home_top"))
             (pad 3 smd rect (at 0 3.5 -30) (size 0.2 0.2) (layers F.Cu F.Paste F.Mask) (net 0 ""))
@@
             (fp_text reference "S29" (at 0 0) (layer F.SilkS) (effects (font (size 1.27 1.27) (thickness 0.15))))
             (fp_text value "" (at 0 0) (layer F.SilkS) hide (effects (font (size 1.27 1.27) (thickness 0.15))))
-            (pad 1 smd rect (at 0 1.5 -30) (size 0.2 0.2) (layers F.Cu F.Paste F.Mask) (net 21 "P5"))
+            (pad 1 smd rect (at 0 1.5 -30) (size 0.2 0.2) (layers F.Cu F.Paste F.Mask) (net 26 "P4"))
             (pad 2 smd rect (at 0 2.5 -30) (size 0.2 0.2) (layers F.Cu F.Paste F.Mask) (net 35 "far_top"))
             (pad 3 smd rect (at 0 3.5 -30) (size 0.2 0.2) (layers F.Cu F.Paste F.Mask) (net 0 ""))
